Commit message: update 10.10添加防爆

File: aprilTag-ros2/src/robot_model/z1_v1.0/urdf/z1_v1.urdf (robot description, URDF)
Before this commit: robot z1_v1, 31 links, 30 joints
Links:
- added link arm_base_link_visual, mass 0.001
Joints:
- added joint arm_base_link_visual: type continuous, parent arm_base_link, child arm_base_link_visual, origin xyz=0.0 0 0 rpy=0 0 0
